Commit message: Update

File: src/dvrk-ros/dvrk_model/model/MTM.urdf.xacro (robot description, xacro)
@@ -501,5 +501,5 @@
       <type>transmission_interface/SimpleTransmission</type>
       <joint name="wrist_platform">
-        <hardwareInterface>EffortJointInterface</hardwareInterface>
+        <hardwareInterface>hardware_interface/EffortJointInterface</hardwareInterface>
       </joint>
       <actuator name="motor4">
@@ -511,5 +511,5 @@
       <type>transmission_interface/SimpleTransmission</type>
       <joint name="wrist_pitch">
-        <hardwareInterface>EffortJointInterface</hardwareInterface>
+        <hardwareInterface>hardware_interface/EffortJointInterface</hardwareInterface>
       </joint>
       <actuator name="motor5">
@@ -521,5 +521,5 @@
       <type>transmission_interface/SimpleTransmission</type>
       <joint name="wrist_yaw">
-        <hardwareInterface>EffortJointInterface</hardwareInterface>
+        <hardwareInterface>hardware_interface/EffortJointInterface</hardwareInterface>
       </joint>
       <actuator name="motor6">

File: src/dvrk-ros/dvrk_model/model/dvrk_psm.base.urdf.xacro (robot description, xacro)
@@ -183,6 +183,6 @@
       <mass value="0.1"/>
       <inertia
-        ixx="0.1" ixy="0.0" ixz="0.0"
-        iyy="0.1" iyz="0.0"
+        ixx="0.001" ixy="0.0" ixz="0.0"
+        iyy="0.001" iyz="0.0"
         izz="0.005"/>
     </inertial>
@@ -218,6 +218,6 @@
     <joint name="${prefix}outer_insertion_joint" type="prismatic">
       <!-- <parent link="${prefix}outer_insertion_link"/> -->
-      <!-- <parent link="${prefix}psm_base_link"/> -->
-      <parent link="${prefix}outer_pitch_link"/>
+      <parent link="${prefix}psm_base_link"/>
+      <!-- <parent link="${prefix}outer_pitch_link"/>-->
       <child link="${prefix}tool_main_link"/>
       <axis xyz="0 0 1"/>
@@ -238,6 +238,6 @@
       <mass value="0.1"/>
       <inertia
-        ixx="0.1" ixy="0.0" ixz="0.0"
-        iyy="0.1" iyz="0.0"
+        ixx="0.001" ixy="0.0" ixz="0.0"
+        iyy="0.001" iyz="0.0"
         izz="0.005"/>
       </inertial>
@@ -296,5 +296,5 @@
     <type>transmission_interface/SimpleTransmission</type>
     <joint name="${prefix}outer_yaw_joint">
-      <hardwareInterface>EffortJointInterface</hardwareInterface>
+	<hardwareInterface>hardware_interface/EffortJointInterface</hardwareInterface>
     </joint>
     <actuator name="${prefix}motor1">
@@ -306,5 +306,5 @@
     <type>transmission_interface/SimpleTransmission</type>
     <joint name="${prefix}outer_pitch_joint">
-      <hardwareInterface>EffortJointInterface</hardwareInterface>
+        <hardwareInterface>hardware_interface/EffortJointInterface</hardwareInterface>
     </joint>
     <actuator name="${prefix}motor2">
@@ -316,5 +316,5 @@
     <type>transmission_interface/SimpleTransmission</type>
     <joint name="${prefix}outer_pitch_joint_1">
-      <hardwareInterface>EffortJointInterface</hardwareInterface>
+        <hardwareInterface>hardware_interface/EffortJointInterface</hardwareInterface>
     </joint>
     <actuator name="${prefix}motor2_1">
@@ -326,5 +326,5 @@
     <type>transmission_interface/SimpleTransmission</type>
     <joint name="${prefix}outer_pitch_joint_2">
-      <hardwareInterface>EffortJointInterface</hardwareInterface>
+        <hardwareInterface>hardware_interface/EffortJointInterface</hardwareInterface>
     </joint>
     <actuator name="${prefix}motor2_2">
@@ -336,5 +336,5 @@
     <type>transmission_interface/SimpleTransmission</type>
     <joint name="${prefix}outer_pitch_joint_3">
-      <hardwareInterface>EffortJointInterface</hardwareInterface>
+        <hardwareInterface>hardware_interface/EffortJointInterface</hardwareInterface>
     </joint>
     <actuator name="${prefix}motor2_3">
@@ -346,5 +346,5 @@
     <type>transmission_interface/SimpleTransmission</type>
     <joint name="${prefix}outer_pitch_joint_4">
-      <hardwareInterface>EffortJointInterface</hardwareInterface>
+        <hardwareInterface>hardware_interface/EffortJointInterface</hardwareInterface>
     </joint>
     <actuator name="${prefix}motor2_4">
@@ -356,5 +356,5 @@
     <type>transmission_interface/SimpleTransmission</type>
     <joint name="${prefix}outer_pitch_joint_5">
-      <hardwareInterface>EffortJointInterface</hardwareInterface>
+        <hardwareInterface>hardware_interface/EffortJointInterface</hardwareInterface>
     </joint>
     <actuator name="${prefix}motor2_5">
@@ -366,5 +366,5 @@
     <type>transmission_interface/SimpleTransmission</type>
     <joint name="${prefix}outer_insertion_joint">
-      <hardwareInterface>EffortJointInterface</hardwareInterface>
+        <hardwareInterface>hardware_interface/EffortJointInterface</hardwareInterface>
     </joint>
     <actuator name="${prefix}motor3">
@@ -376,5 +376,5 @@
     <type>transmission_interface/SimpleTransmission</type>
     <joint name="${prefix}outer_roll_joint">
-      <hardwareInterface>EffortJointInterface</hardwareInterface>
+        <hardwareInterface>hardware_interface/EffortJointInterface</hardwareInterface>
     </joint>
     <actuator name="${prefix}motor4">
